Commit message: Moved urdf to package and added cmake rules to create SICK.urdf at build

File: lab_5_ws/src/drive_jackal/urdf/sick_lms291.urdf.xacro (robot description, xacro)
@@ -12,7 +12,7 @@
     </inertial>
     <visual>
-      <origin xyz="0 0 0.0925" rpy="0 0 0" />
+      <origin xyz="0 0 0" rpy="0 0 0" />
       <geometry>
-        <box size="0.155 0.156 0.185"/>
+        <mesh filename="package://drive_jackal/mesh/lms291_asm.stl"/>
       </geometry>
       <material name="white">

Commit message: Updated urdf to include mount and updated the placement

File: lab_5_ws/src/drive_jackal/urdf/sick_lms291.urdf.xacro (robot description, xacro)
@@ -1,4 +1,11 @@
 <?xml version="1.0"?>
 <robot xmlns:xacro="http://ros.org/wiki/xacro" name="lms291_lrf">
+  <xacro:property name="PI" value="3.1415926535897931" />
+  <material name="white">
+    <color rgba="1 1 1 1"/>
+  </material>
+  <material name="blue">
+    <color rgba="0 0 .8 1"/>
+  </material>
   <!-- LMS291 Lidar model -->
   <link name="lms291">
@@ -12,14 +19,11 @@
     </inertial>
     <visual>
-      <origin xyz="0 0 0" rpy="0 0 0" />
       <geometry>
-        <mesh filename="package://drive_jackal/mesh/lms291_asm.stl"/>
+        <mesh filename="package://drive_jackal/mesh/lms291_asm.stl" scale="0.001 0.001 0.001"/>
       </geometry>
-      <material name="white">
-        <color rgba="1 1 1 1"/>
-      </material>
+      <material name="white"/>
     </visual>
     <collision>
-      <origin xyz="0 0 0.0925" rpy="0 0 0" />
+      <origin xyz="0 0 0" rpy="0 0 0" />
       <geometry>
         <box size="0.155 0.156 0.185"/>
@@ -27,8 +31,38 @@
     </collision>
   </link>
-  <!-- Link for LMS291 to Jackal -->
-  <joint name="lms291_mount" type="fixed">
+  <!-- LMS291 Lidar Mount model -->
+  <link name="lms291_mount">
+    <inertial>
+      <mass value="0.4" />
+      <origin xyz="0 0 0" />
+      <inertia
+      ixx="0.0" ixy="0.0" ixz="0.0"
+      iyy="0.0" iyz="0.0"
+      izz="0.0"/>
+    </inertial>
+    <visual>
+      <geometry>
+        <mesh filename="package://drive_jackal/mesh/LidarMount.stl" scale="0.001 0.001 0.001"/>
+      </geometry>
+      <material name="blue"/>
+    </visual>
+    <collision>
+      <origin xyz="0 0 0.0925" rpy="${PI} 0 0" />
+      <geometry>
+        <box size="0.155 0.156 0.185"/>
+      </geometry>
+    </collision>
+  </link>
+  <!-- Link for LMS291 to Mount -->
+  <joint name="lms291_to_mount" type="fixed">
+    <origin xyz="0 -0.093 0.078" rpy="0 0 ${PI/2}" />
+    <parent link="lms291_mount"/>
+    <child link="lms291"/>
+  </joint>
+  <!-- Link for Mount to Jackal -->
+  <joint name="lms291_mount_to_jackal" type="fixed">
+    <origin xyz="-0.090 0 0" rpy="0 0 ${PI/2}" />
     <parent link="front_mount"/>
-    <child link="lms291"/>
+    <child link="lms291_mount"/>
   </joint>
   <gazebo reference="lms291">

Commit message: Added lidar test launch and a link for lidar data

File: lab_5_ws/src/drive_jackal/urdf/sick_lms291.urdf.xacro (robot description, xacro)
@@ -2,9 +2,9 @@
 <robot xmlns:xacro="http://ros.org/wiki/xacro" name="lms291_lrf">
   <xacro:property name="PI" value="3.1415926535897931" />
-  <material name="white">
-    <color rgba="1 1 1 1"/>
+  <material name="blue">
+    <color rgba="0 0 1 1"/>
   </material>
-  <material name="blue">
-    <color rgba="0 0 .8 1"/>
+  <material name="grey">
+    <color rgba=".3 .3 .3 1.0"/>
   </material>
   <!-- LMS291 Lidar model -->
@@ -22,5 +22,5 @@
         <mesh filename="package://drive_jackal/mesh/lms291_asm.stl" scale="0.001 0.001 0.001"/>
       </geometry>
-      <material name="white"/>
+      <material name="blue"/>
     </visual>
     <collision>
@@ -45,5 +45,5 @@
         <mesh filename="package://drive_jackal/mesh/LidarMount.stl" scale="0.001 0.001 0.001"/>
       </geometry>
-      <material name="blue"/>
+      <material name="grey"/>
     </visual>
     <collision>
@@ -54,4 +54,11 @@
     </collision>
   </link>
+  <link name="lms291_data"/>
+  <!-- Link for Scan data to LMS291 -->
+  <joint name="scan_to_lms291" type="fixed">
+    <origin xyz="0 0 0" rpy="0 0 ${PI}" />
+    <parent link="lms291"/>
+    <child link="lms291_data"/>
+  </joint>
   <!-- Link for LMS291 to Mount -->
   <joint name="lms291_to_mount" type="fixed">
@@ -67,4 +74,5 @@
   </joint>
   <gazebo reference="lms291">
+    <material>Gazebo/Blue</material>
     <turnGravityOff>true</turnGravityOff>
     <sensor type="ray" name="lms291">
@@ -98,3 +106,6 @@
     </sensor>
   </gazebo>
+  <gazebo reference="lms291_mount">
+    <material>Gazebo/Grey</material>
+  </gazebo>
 </robot>

Commit message: Updated reference frame for lidar data

File: lab_5_ws/src/drive_jackal/urdf/sick_lms291.urdf.xacro (robot description, xacro)
@@ -54,5 +54,24 @@
     </collision>
   </link>
-  <link name="lms291_data"/>
+  <link name="lms291_data">
+    <inertial>
+      <mass value="0.00001" />
+      <origin xyz="0 0 0" />
+      <inertia
+      ixx="0.00001" ixy="0.0" ixz="0.0"
+      iyy="0.00001" iyz="0.0"
+      izz="0.00001"/>
+    </inertial>
+    <visual>
+      <geometry>
+        <sphere radius="0.00001"/>
+      </geometry>
+    </visual>
+    <collision>
+      <geometry>
+        <sphere radius="0.00001"/>
+      </geometry>
+    </collision>
+  </link>
   <!-- Link for Scan data to LMS291 -->
   <joint name="scan_to_lms291" type="fixed">
